Commit message: rotate 3d lidar by 90 degrees
Signed-off-by: mitsudome-r <ryohsuke.mitsudome@tier4.jp>

File: nova_carter_description/urdf/nova_carter.urdf.xacro (robot description, xacro)
@@ -53,5 +53,5 @@
   <!-- 3D LIDAR -->
   <xacro:pandar_xt32_lidar name="front" parent="base_link">
-    <origin xyz="-0.231700 0.0 0.526300" rpy="0.0 0.0 0.0"/>
+    <origin xyz="-0.231700 0.0 0.526300" rpy="0.0 0.0 ${M_PI/2}"/>
   </xacro:pandar_xt32_lidar>
   <!-- 2D LIDARs -->
